File: V2/ESP-pwm-4ch-V2.kicad_pcb (KiCad board)
At the start: 2 copper layers, 103 x 67.8 mm, 38 parts, among them J1 12VDC, J2 OUT1, J3 OUT2, J4 OUT3, J5 OUT4, Q1 IRLB8721PBF, Q2 IRLB8721PBF, Q3 IRLB8721PBF, Q4 IRLB8721PBF, U1 L78M05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

Commit message: Updated connectors
Parts:
- removed REF**: OSHW-Logo2_14.6x12mm_SilkScreen, Symbol:OSHW-Logo2_14.6x12mm_SilkScreen
- Q1, Q2, Q3, Q4: footprint Tales:TO-220-3_Vertical -> Package_TO_SOT_THT:TO-220-3_Vertical
- U2: footprint Tales:WEMOS_D1_mini_light_pads -> Module:WEMOS_D1_mini_light
- U3: footprint Tales:Olimex_ESP32-POE_Pads -> Tales:Olimex_ESP32-POE
Connections:
- net +3V3 renamed +3.3V
Routing:
- net GNDREF: track 328.4 -> 327.3 mm
