File: V2/ESP-pwm-4ch-V2.kicad_sch (KiCad schematic)
At the start: 33 parts

Commit message: Kicad version update
Parts:
- C1: value (none) -> 47uF/35V/6,3x5,4; footprint (none) -> Tales:CP_Elec_6.3x5.4
- C2: value (none) -> 0,33uF/35V; footprint (none) -> Tales:CP_EIA-3216-18_Kemet-A_Pad1.58x1.35mm_HandSolder
- C3, C4, C6: value (none) -> 0,1uF/50V/0805; footprint (none) -> Tales:C_0805_2012Metric
- C5, C7: value (none) -> 1uF 35V; footprint (none) -> Tales:CP_EIA-3216-18_Kemet-A_Pad1.58x1.35mm_HandSolder
- D1: value (none) -> SM4007PL/SOD-123; footprint (none) -> Tales:D_SOD-123
- D2, D3, D4: value (none) -> GREEN/0603; footprint (none) -> Tales:LED_0603_1608Metric
- J1: value (none) -> 12VDC; footprint (none) -> Tales:TerminalBlock_Phoenix_MKDS-3-2-5.08_1x02_P5.08mm_Horizontal
- J2: value (none) -> OUT1; footprint (none) -> Tales:TerminalBlock_Phoenix_MKDS-3-2-5.08_1x02_P5.08mm_Horizontal
- J3: value (none) -> OUT2; footprint (none) -> Tales:TerminalBlock_Phoenix_MKDS-3-2-5.08_1x02_P5.08mm_Horizontal
- J4: value (none) -> OUT3; footprint (none) -> Tales:TerminalBlock_Phoenix_MKDS-3-2-5.08_1x02_P5.08mm_Horizontal
- J5: value (none) -> OUT4; footprint (none) -> Tales:TerminalBlock_Phoenix_MKDS-3-2-5.08_1x02_P5.08mm_Horizontal
- Q1, Q2, Q3, Q4: value (none) -> IRLB8721PBF; footprint (none) -> Tales:TO-220-3_Vertical
- R1: value (none) -> 2k2/0,125W/0805; footprint (none) -> Tales:R_0805_2012Metric
- R2: value (none) -> 680R/0,125W/0805; footprint (none) -> Tales:R_0805_2012Metric
- R3: value (none) -> 270R/0,125W/0805; footprint (none) -> Tales:R_0805_2012Metric
- R4, R5, R6, R7: value (none) -> 22R/0,125W/0805; footprint (none) -> Tales:R_0805_2012Metric
- R8: value (none) -> 4k7/0,125W/0805; footprint (none) -> Tales:R_0805_2012Metric
- U1: value (none) -> L78M05; footprint (none) -> Tales:TO-252-2
- U2: value (none) -> WeMos_D1_mini; footprint (none) -> Tales:WEMOS_D1_mini_light_pads
- U3: value (none) -> Olimex_ESP32-POE; footprint (none) -> Tales:Olimex_ESP32-POE_Pads
- U4, U5: value (none) -> IR4427; footprint (none) -> Tales:SOIC-8_3.9x4.9mm_P1.27mm

Commit message: Updated connectors
Parts:
- Q1, Q2, Q3, Q4: footprint Tales:TO-220-3_Vertical -> Package_TO_SOT_THT:TO-220-3_Vertical
- U2: footprint Tales:WEMOS_D1_mini_light_pads -> Module:WEMOS_D1_mini_light
- U3: footprint Tales:Olimex_ESP32-POE_Pads -> Tales:Olimex_ESP32-POE
Connections:
- net +3V3 renamed +3.3V
Changed lines of the file:
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@@
+      (effects (font (size 1.27 1.27)) hide)
+    )
+    (property "Sim.Device" "D" (at 53.34 34.29 0)
+      (effects (font (size 1.27 1.27)) hide)
+    )
+    (property "Sim.Pins" "1=K 2=A" (at 53.34 34.29 0)
       (effects (font (size 1.27 1.27)) hide)
     )
@@
       (effects (font (size 1.27 1.27)) (justify left))
     )
-    (property "Footprint" "Tales:Olimex_ESP32-POE_Pads" (at 186.69 189.23 0)
+    (property "Footprint" "Tales:Olimex_ESP32-POE" (at 186.69 189.23 0)
       (effects (font (size 1.27 1.27)) hide)
     )
@@
       (effects (font (size 1.27 1.27)) (justify left))
     )
-    (property "Footprint" "Tales:WEMOS_D1_mini_light_pads" (at 186.69 128.27 0)
+    (property "Footprint" "Module:WEMOS_D1_mini_light" (at 186.69 128.27 0)
       (effects (font (size 1.27 1.27)) hide)
     )
@@
       (effects (font (size 1.27 1.27)) (justify left))
     )
-    (property "Footprint" "Tales:TO-220-3_Vertical" (at 350.52 93.345 0)
+    (property "Footprint" "Package_TO_SOT_THT:TO-220-3_Vertical" (at 350.52 93.345 0)
       (effects (font (size 1.27 1.27) italic) (justify left) hide)
     )
@@
       (effects (font (size 1.27 1.27)) (justify left))
     )
-    (property "Footprint" "Tales:TO-220-3_Vertical" (at 350.52 132.715 0)
+    (property "Footprint" "Package_TO_SOT_THT:TO-220-3_Vertical" (at 350.52 132.715 0)
       (effects (font (size 1.27 1.27) italic) (justify left) hide)
     )
@@
       (effects (font (size 1.27 1.27)) (justify left))
     )
-    (property "Footprint" "Tales:TO-220-3_Vertical" (at 350.52 173.355 0)
+    (property "Footprint" "Package_TO_SOT_THT:TO-220-3_Vertical" (at 350.52 173.355 0)
       (effects (font (size 1.27 1.27) italic) (justify left) hide)
     )
@@
       (effects (font (size 1.27 1.27)) (justify left))
     )
-    (property "Footprint" "Tales:TO-220-3_Vertical" (at 350.52 51.435 0)
+    (property "Footprint" "Package_TO_SOT_THT:TO-220-3_Vertical" (at 350.52 51.435 0)
       (effects (font (size 1.27 1.27) italic) (justify left) hide)
     )
